File: meshtonic/meshtonic/meshtonic.kicad_pcb (KiCad board)
At the start: 6 copper layers, 133 x 110 mm, 122 parts, among them J1 GROVE-CONNECTOR-DIP_4P-2.0_, J10 U.FL, J11 U.FL, J13 Header 1x7 2.54mm, J14 Header 1x7 2.54mm, J15 Header 1x7 2.54mm, J16 Header 1x7 2.54mm, J18 Micro_SD_Card_passive_clk, J19 Conn_02x06_Top_Bottom, J2 GROVE-CONNECTOR-DIP_4P-2.0_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

Commit message: adds silkscreens init
Parts:
- added G***: LOGO, Graphics:astronaut_small, F.Cu at (146.1, 89.9)
- added G***: LOGO, LOGO, F.Cu at (148.3, 113.2)
Routing:
- removed copper zone on B.Cu, net GND
