File: pcb/Sensors.kicad_sch (KiCad schematic)
At the start: 18 parts, among them U4 TCA9548APWR

Commit message: fixes SCL to SDA on J_AS1
Connections:
- net I2C_SCL: no longer J_AS1.2 (Pin_2), R13.2
- net I2C_SDA: now also J_AS1.2 (Pin_2), R13.2
Changed lines of the file:
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@@
 		)
 	)
-	(global_label "I2C_SCL"
+	(global_label "I2C_SDA"
 		(shape input)
 		(at 111.76 138.43 180)
@@
 		)
 		(property "Intersheetrefs" "${INTERSHEET_REFS}"
-			(at 101.2153 138.43 0)
+			(at 101.1548 138.43 0)
 			(show_name no)
 			(do_not_autoplace no)
