File: pcb/meshtonic_h4m_v2.kicad_pcb (KiCad board)
At the start: 6 copper layers, 71.1 x 168.4 mm, 117 parts, among them J1 GROVE-CONNECTOR-DIP_4P-2.0_, J10 Conn_01x02, J11 Conn_01x02, J12 JST_2mm_LiPo, J13 Screw_Terminal_01x02, J14 Micro_SD_Card_passive_clk, J15 H4M_2x6_MDK, J2 GROVE-CONNECTOR-DIP-90D_4P-2.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, J3 GROVE-CONNECTOR-DIP_4P-2.0_, J4 GROVE-CONNECTOR-DIP_4P-2.0_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

Commit message: solves some issues
Routing:
- net LORA_RST: track 171.3 -> 168.9 mm
- net UART0_RX: track 130.7 -> 129.6 mm
- net GND: track 77.2 -> 77.9 mm
- net I2C_SDA: track 225.2 -> 224.6 mm
