File: pcb/meshtonic_h4m_v2.kicad_pcb (KiCad board)
At the start: 6 copper layers, 71.1 x 168.4 mm, 117 parts, among them J1 GROVE-CONNECTOR-DIP_4P-2.0_, J10 Conn_01x02, J11 Conn_01x02, J12 JST_2mm_LiPo, J13 Screw_Terminal_01x02, J14 Micro_SD_Card_passive_clk, J15 H4M_2x6_MDK, J2 GROVE-CONNECTOR-DIP-90D_4P-2.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, J3 GROVE-CONNECTOR-DIP_4P-2.0_, J4 GROVE-CONNECTOR-DIP_4P-2.0_, J5 GROVE-CONNECTOR-DIP_4P-2.0_, J6 GROVE-CONNECTOR-DIP_4P-2.0_, J7 GROVE-CONNECTOR-DIP_4P-2.0_, J8 GROVE-CONNECTOR-SMD_4+2P-2.0_, J9 Conn_01x02, U1 TPS63020DSJR, U2 CN3170, U3 XIAO-S3-Plus, U4 TCA9548APWR, U5 MCP23017x-x-SS

Commit message: adds a resistor between TMP and GND in Power sheet to allow battery charging
Parts:
- added R45: 10k, PCM_SparkFun-Resistor:R_0603_1608Metric, F.Cu at (158.9, 15.5)
- moved D5 13.2 mm to (156.5, 27.3)
- moved R5 10.8 mm to (155.0, 15.4), turned to -90 degrees
- moved R3 10.2 mm to (159.3, 26.7), turned to 180 degrees
- moved R2 4.91 mm to (162.8, 15.9), turned to 90 degrees
- moved D4 2.99 mm to (158.9, 19.9), turned to 90 degrees
- moved ST3 1.73 mm to (158.5, 33.6)
- moved JP_H4M_3V1 1.50 mm to (166.5, 21.5)
- moved JP_VBAT_H4M1 1.50 mm to (162.9, 21.5)
- moved C2 0.96 mm to (151.6, 15.0), turned to -90 degrees
Connections:
- U2 pad 1: GND -> Net-(U2-TEMP)
Routing:
- net Net-(U2-ISET): track 30.2 -> 2.15 mm
- net Net-(D5-K): track 23.7 -> 4.69 mm
- net Net-(D4-K): track 19.2 -> 8.39 mm
- net GND: track 77.9 -> 83.1 mm
- net Net-(U2-TEMP): track 0.00 -> 3.35 mm
- net Net-(D4-A): track 2.63 -> 5.25 mm
- net VBAT_H4M: track 34.5 -> 32.2 mm
- net VBAT: track 380.9 -> 378.8 mm
- net Net-(D5-A): track 2.16 -> 2.82 mm
